Commit message: Add D435 camera

File: piper_description/urdf/piper_description.urdf (robot description, URDF)
Before this commit: robot piper, 10 links, 9 joints
Links:
- link link2: mass 1.16 -> 1.17
- link link5: mass 0.39 -> 0.383
- link link6: mass 0.46 -> 0.00699089613564366
Joints:
- joint joint1: limit lower=-2.618 upper=2.618 effort=100 velocity=5 -> lower=-2.618 upper=2.168 effort=100 velocity=5

File: piper_description/urdf/piper_description_old.urdf (robot description, URDF)
Before this commit: robot piper, 10 links, 9 joints
Links:
- link link2: mass 1.16 -> 1.17
- link link5: mass 0.39 -> 0.383
- link link6: mass 0.46 -> 0.00699089613564366
Joints:
- joint joint1: limit lower=-2.618 upper=2.618 effort=100 velocity=5 -> lower=-2.618 upper=2.168 effort=100 velocity=5

File: piper_description/urdf/piper_no_gripper_description.urdf (robot description, URDF)
Before this commit: robot piper, 7 links, 6 joints
Links:
- link link2: mass 1.16 -> 1.17
- link link5: mass 0.39 -> 0.383
- link link6: mass 0.46 -> 0.00699089613564366
Joints:
- joint joint1: limit lower=-2.618 upper=2.618 effort=100 velocity=5 -> lower=-2.618 upper=2.168 effort=100 velocity=5

File: piper_description/urdf/piper_no_gripper_description_old.urdf (robot description, URDF)
Before this commit: robot piper, 7 links, 6 joints
Links:
- link link2: mass 1.16 -> 1.17
- link link5: mass 0.39 -> 0.383
- link link6: mass 0.46 -> 0.00699089613564366
Joints:
- joint joint1: limit lower=-2.618 upper=2.618 effort=100 velocity=5 -> lower=-2.618 upper=2.168 effort=100 velocity=5
