Commit message: add piper_l piper_x piper_h urdf and USD

File: piper_x_description/urdf/piper_x_description_d435.urdf (robot description, URDF)
Before this commit: robot piper_x_camera, 13 links, 12 joints
Links:
- link Link7: mass 0.0 -> 0.0264822021416248
- link camera_link: geometry collision box size=0.02505 0.09 0.025; visual mesh filename=package://realsense2_description/meshes/d435.dae
